Commit message: updated params

File: turtlebot3_description/urdf/turtlebot3_teleops.gazebo.xacro (robot description, xacro)
@@ -124,6 +124,6 @@
         <cameraName>camera</cameraName>
         <frameName>camera_rgb_optical_frame</frameName>
-        <imageTopicName>rgb/image_raw</imageTopicName>
-        <cameraInfoTopicName>rgb/camera_info</cameraInfoTopicName>
+        <imageTopicName>image_raw</imageTopicName>
+        <cameraInfoTopicName>camera_info</cameraInfoTopicName>
         <hackBaseline>0.07</hackBaseline>
         <distortionK1>0.0</distortionK1>
@@ -137,6 +137,6 @@
   <!-- Adding the kinect sensor -->
   <xacro:include filename="$(find kinect_v2)/urdf/kinect_v2.urdf.xacro" />
-  <xacro:kinect_v2  parent="base_link">
-    <origin xyz="-0.05 0 0.1" rpy="0 0 0"/>
+  <xacro:kinect_v2 parent="base_link">
+    <origin xyz="-0.05 0 0.15" rpy="0 0 0"/>
   </xacro:kinect_v2>
   <!-- Adding the GPS sensor -->
@@ -154,3 +154,35 @@
     </plugin>
   </gazebo>
+  <!--gazebo reference="base_scan">
+    <material>Gazebo/FlatBlack</material>
+    <sensor type="ray" name="lds_lfcd_sensor">
+      <pose>0 0 0 0 0 0</pose>
+      <visualize>$(arg laser_visual)</visualize>
+      <update_rate>5</update_rate>
+      <ray>
+        <scan>
+          <horizontal>
+            <samples>360</samples>
+            <resolution>1</resolution>
+            <min_angle>0.0</min_angle>
+            <max_angle>6.28319</max_angle>
+          </horizontal>
+        </scan>
+        <range>
+          <min>0.120</min>
+          <max>3.5</max>
+          <resolution>0.015</resolution>
+        </range>
+        <noise>
+          <type>gaussian</type>
+          <mean>0.0</mean>
+          <stddev>0.01</stddev>
+        </noise>
+      </ray>
+      <plugin name="gazebo_ros_lds_lfcd_controller" filename="libgazebo_ros_laser.so">
+        <topicName>scan</topicName>
+        <frameName>base_scan</frameName>
+      </plugin>
+    </sensor>
+  </gazebo-->
 </robot>

File: turtlebot3_description/urdf/turtlebot3_teleops.urdf.xacro (robot description, xacro)
@@ -174,5 +174,5 @@
   </link>
   <joint name="camera_rgb_joint" type="fixed">
-    <origin xyz="0.003 0.011 0.009" rpy="0 0 0"/>
+    <origin xyz="0.003 0.011 0.009" rpy="3.14 0 0"/>
     <parent link="camera_link"/>
     <child link="camera_rgb_frame"/>

File: turtlebot3_description/urdf/turtlebot3_waffle_pi.gazebo.xacro (robot description, xacro)
@@ -134,5 +134,5 @@
     </sensor>
   </gazebo>
-<!--link : https://www.raspberrypi.org/documentation/hardware/camera/-->
+  <!--link : https://www.raspberrypi.org/documentation/hardware/camera/-->
   <gazebo reference="camera_rgb_frame">
     <sensor type="camera" name="Pi Camera">

Commit message: exchanged gps module for teleops

File: turtlebot3_description/urdf/turtlebot3_teleops.gazebo.xacro (robot description, xacro)
@@ -58,6 +58,7 @@
       <odometryFrame>odom</odometryFrame>
       <odometrySource>world</odometrySource>
-      <publishOdomTF>true</publishOdomTF>
-      <robotBaseFrame>base_footprint</robotBaseFrame>
+      <robotBaseFrame>base_link</robotBaseFrame>
+      <!--robotBaseFrame>base_footprint</robotBaseFrame-->
+      <publishOdomTF>false</publishOdomTF>
       <publishWheelTF>false</publishWheelTF>
       <publishTf>true</publishTf>
@@ -79,5 +80,5 @@
       <bodyName>imu_link</bodyName>
       <frameName>imu_link</frameName>
-      <topicName>imu</topicName>
+      <topicName>imu/data</topicName>
       <serviceName>imu_service</serviceName>
       <gaussianNoise>0.0</gaussianNoise>
@@ -141,9 +142,10 @@
   </xacro:kinect_v2-->
   <!-- Adding the GPS sensor -->
-  <gazebo>
+  <!--gazebo reference="gps_link">
     <plugin name="gps_controller" filename="libhector_gazebo_ros_gps.so">
       <alwayson>true</alwayson>
       <updaterate>1.0</updaterate>
       <bodyname>base_link</bodyname>
+      <framename>gps_link</framename>
       <topicname>/fix</topicname>
       <velocitytopicname>/fix_velocity</velocitytopicname>
@@ -152,4 +154,19 @@
       <velocitydrift>0 0 0</velocitydrift>
       <velocitygaussiannoise>0.1 0.1 0.1</velocitygaussiannoise>
+    </plugin>
+  </gazebo-->
+  <gazebo>
+    <plugin name="gps_controller" filename="libhector_gazebo_ros_gps.so">
+      <!--robotNamespace>$(arg robot_namespace)</robotNamespace-->
+      <updateRate>40</updateRate>
+      <bodyName>base_link</bodyName>
+      <frameId>base_link</frameId>
+      <topicName>navsat/fix</topicName>
+      <velocityTopicName>navsat/vel</velocityTopicName>
+      <referenceLatitude>49.9</referenceLatitude>
+      <referenceLongitude>8.9</referenceLongitude>
+      <referenceHeading>0</referenceHeading>
+      <referenceAltitude>0</referenceAltitude>
+      <drift>0.0001 0.0001 0.0001</drift>
     </plugin>
   </gazebo>

File: turtlebot3_description/urdf/turtlebot3_teleops.urdf.xacro (robot description, xacro)
@@ -3,10 +3,10 @@
   <xacro:include filename="$(find turtlebot3_description)/urdf/common_properties.xacro"/>
   <xacro:include filename="$(find turtlebot3_description)/urdf/turtlebot3_teleops.gazebo.xacro"/>
-  <link name="base_footprint"/>
+  <!--link name="base_footprint"/>
   <joint name="base_joint" type="fixed">
     <parent link="base_footprint"/>
     <child link="base_link" />
     <origin xyz="0 0 0.010" rpy="0 0 0"/>
-  </joint>
+  </joint-->
   <link name="base_link">
     <visual>
@@ -31,4 +31,10 @@
     </inertial>
   </link>
+  <link name="base_footprint"/>
+  <joint name="base_footprint_joint" type="fixed">
+    <origin xyz="0 0 0.010" rpy="0 0 0"/>
+    <parent link="base_link"/>
+    <child link="base_footprint" />
+  </joint>
   <joint name="wheel_left_joint" type="continuous">
     <parent link="base_link"/>
@@ -185,3 +191,9 @@
   </joint>
   <link name="camera_rgb_optical_frame"/>
+  <joint name="gps_joint" type="fixed">
+    <parent link="base_link"/>
+    <child link="gps_link"/>
+    <origin xyz="0.15 0 0.15" rpy="0 0 0"/>
+  </joint>
+  <link name="gps_link"/>
 </robot>
